File: EMG circuit/mumai.brd (EAGLE design)
At the start: 46.3 x 35.2 mm, 64 parts, among them IC1 MCP1703DB, J1 AUDIO-JACK2SMD, U1 INA333AIDGKR, U2 OPA2211AIDDA, U3 OPA2211AIDDA, U4 OPA2211AIDDA, U5 OPA2211AIDDA, U6 OPA2211AIDDA, U7 REF3125AIDBZT

Commit message: Update EMG board
Parts:
- removed U$1: (no value), new_bq:BQ_LOGO
Changed lines of the file:
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@@
 <?xml version="1.0" encoding="utf-8"?>
 <!DOCTYPE eagle SYSTEM "eagle.dtd">
-<eagle version="7.4.0">
+<eagle version="7.5.0">
 <drawing>
 <settings>
@@
 <attribute name="VALUE" x="41.021" y="20.2565" size="0.4064" layer="27" rot="R90"/>
 </element>
-<element name="U$1" library="new_bq" package="BQ_LOGO" value="" x="28.829" y="11.938" smashed="yes" rot="MR0"/>
 </elements>
 <signals>
